Commit message: improved urdf

File: spider.urdf (robot description, URDF)
Before this commit: robot spider, 7 links, 6 joints
Links:
- link body: geometry collision cylinder length=0.05 radius=0.1; visual cylinder length=0.05 radius=0.1
- link shin_leg1: geometry collision box size=0.2 0.05 0.05; visual box size=0.2 0.05 0.05
- link shin_leg2: geometry collision box size=0.2 0.05 0.05; visual box size=0.2 0.05 0.05
- link shin_leg3: geometry collision box size=0.2 0.05 0.05; visual box size=0.2 0.05 0.05
- link thigh_leg1: geometry collision box size=0.2 0.05 0.05; visual box size=0.2 0.05 0.05
- link thigh_leg2: geometry collision box size=0.2 0.05 0.05; visual box size=0.2 0.05 0.05
- link thigh_leg3: geometry collision box size=0.2 0.05 0.05; visual box size=0.2 0.05 0.05
Joints:
- joint hip_joint_leg1: origin xyz=0.1 0 0 rpy=0 0 0 -> xyz=0.1 0 0 rpy=0 1.5708 0
- joint hip_joint_leg2: origin xyz=0.1 0 0 rpy=0 0 2.0944 -> xyz=-0.05 0.0866 0 rpy=0 1.5708 2.0944
- joint hip_joint_leg3: origin xyz=0.1 0 0 rpy=0 0 4.18879 -> xyz=-0.05 -0.0866 0 rpy=0 1.5708 4.18879
